Commit message: update floating cams

File: src/auracle/description/robot_core.xacro (robot description, xacro)
@@ -43,5 +43,5 @@
     <link name="chassis">
         <visual>
-            <origin xyz="${chassis_length/2} 0 0"/>
+            <origin xyz="${chassis_length/2} 0 ${chassis_height/2}"/>
             <geometry>
                 <box size="${chassis_length} ${chassis_width} ${chassis_height}"/>

Commit message: update to match robot_2 params

File: src/auracle/description/robot_core.xacro (robot description, xacro)
@@ -11,5 +11,6 @@
     <xacro:property name="tilted_link" value="0.1"/>
     <xacro:property name="rocker_mass" value="0.5"/>
-    <xacro:property name="wheel_radius" value="0.033"/>
+    <!-- Measured from emmanuel-assembly.stp tire rolling-surface cylinder (was 0.033) -->
+    <xacro:property name="wheel_radius" value="0.0239"/>
     <xacro:property name="wheel_thickness" value="0.026"/>
     <xacro:property name="wheel_mass" value="0.05"/>
